File: Kicad/external_circuits.kicad_sch (KiCad schematic)
At the start: 14 parts

Commit message: working on DSP
Parts:
- gave numbers to parts that had none: 14
Connections:
- net LX renamed Buck_LX
Other:
- moved on the sheet: C11, L3, R3
